Commit message: Move vehicle center in the middle of the wheels

File: simulation_ws/src/sim/description/piracer.xacro (robot description, xacro)
@@ -401,5 +401,5 @@
   <!-- JOINT: chassis -->
   <joint name="chassis_joint" type="fixed">
-    <origin xyz="0 0 0" rpy="0 0 0"/>
+    <origin xyz="-0.1015 0 0" rpy="0 0 0"/>
     <parent link="base_footprint"/>
     <child link="chassis"/>

Commit message: Change frame name base_footprint to base_link

File: simulation_ws/src/sim/description/piracer.xacro (robot description, xacro)
@@ -1,6 +1,6 @@
 <?xml version="1.0"?>
 <robot name="piracer" xmlns:xacro="http://www.ros.org/wiki/xacro">
-  <!-- LINK: base_footprint -->
-  <link name="base_footprint"></link>
+  <!-- LINK: base_link -->
+  <link name="base_link"></link>
   <!-- LINK: chassis -->
   <link name="chassis">
@@ -402,5 +402,5 @@
   <joint name="chassis_joint" type="fixed">
     <origin xyz="-0.1015 0 0" rpy="0 0 0"/>
-    <parent link="base_footprint"/>
+    <parent link="base_link"/>
     <child link="chassis"/>
   </joint>
@@ -539,5 +539,5 @@
       <update_rate>100.0</update_rate>
       <odometry_frame>odom</odometry_frame>
-      <robot_base_frame>base_footprint</robot_base_frame>
+      <robot_base_frame>base_link</robot_base_frame>
       <front_left_joint>front_left_tire_joint</front_left_joint>
       <front_right_joint>front_right_tire_joint</front_right_joint>
@@ -595,5 +595,5 @@
         </ros>
         <camera_name>camera_sensor</camera_name>
-        <frame_name>base_footprint</frame_name>
+        <frame_name>base_link</frame_name>
         <hack_baseline>0.07</hack_baseline>
       </plugin>
